File: ESP8266_arduino.sch (KiCad schematic (older format))
At the start: 2 parts

Commit message: 'rev1'
Parts:
- added R?: 10k, symbol R
- added SW?: SW_Push, symbol SW_Push
Connections:
- net labels added: 3.3V, ADC, CH_PD, GPIO0, GPIO12/MISO, GPIO13/MOSI, GPIO14/SCK, GPIO15, GPIO16, GPIO2, GPIO4/SDA, GPIO5/SCL, RXD, TXD, USB_RX
- wire segments 5 -> 22
Other:
- moved on the sheet: R?, U?
Changed lines of the file:
@@
 LIBS:valves
 LIBS:ESP8266
+LIBS:switches
+LIBS:ESP8266_arduino-cache
 EELAYER 25 0
 EELAYER END
 $Descr A4 11693 8268
 encoding utf-8
-Sheet 1 3
+Sheet 1 4
 Title "Arduino clone using ESP-12E"
 Date ""
@@
 L ESP-12E U?
 U 1 1 589B9F6E
-P 4750 3750
-F 0 "U?" H 4750 3650 50  0000 C CNN
-F 1 "ESP-12E" H 4750 3850 50  0000 C CNN
-F 2 "" H 4750 3750 50  0001 C CNN
-F 3 "" H 4750 3750 50  0001 C CNN
-	1    4750 3750
+P 4700 3300
+F 0 "U?" H 4700 3200 50  0000 C CNN
+F 1 "ESP-12E" H 4700 3400 50  0000 C CNN
+F 2 "" H 4700 3300 50  0001 C CNN
+F 3 "" H 4700 3300 50  0001 C CNN
+	1    4700 3300
 	1    0    0    -1
 $EndComp
@@
 L GND #PWR?
 U 1 1 589BA336
-P 5750 4350
-F 0 "#PWR?" H 5750 4100 50  0001 C CNN
-F 1 "GND" H 5750 4200 50  0000 C CNN
-F 2 "" H 5750 4350 50  0000 C CNN
-F 3 "" H 5750 4350 50  0000 C CNN
-	1    5750 4350
+P 5700 3900
+F 0 "#PWR?" H 5700 3650 50  0001 C CNN
+F 1 "GND" H 5700 3750 50  0000 C CNN
+F 2 "" H 5700 3900 50  0000 C CNN
+F 3 "" H 5700 3900 50  0000 C CNN
+	1    5700 3900
 	1    0    0    -1
 $EndComp
 Wire Wire Line
-	5650 4150 5750 4150
+	5600 3700 5700 3700
 Wire Wire Line
-	5750 4150 5750 4350
+	5700 3700 5700 3900
 $Comp
 L R R?
 U 1 1 589BA5F2
-P 6000 3550
-F 0 "R?" V 6080 3550 50  0000 C CNN
-F 1 "1K" V 6000 3550 50  0000 C CNN
-F 2 "" V 5930 3550 50  0000 C CNN
-F 3 "" H 6000 3550 50  0000 C CNN
-	1    6000 3550
+P 5950 3100
+F 0 "R?" V 6030 3100 50  0000 C CNN
+F 1 "1K" V 5950 3100 50  0000 C CNN
+F 2 "" V 5880 3100 50  0000 C CNN
+F 3 "" H 5950 3100 50  0000 C CNN
+	1    5950 3100
 	0    1    1    0
 $EndComp
 Wire Wire Line
-	5650 3550 5850 3550
+	5600 3100 5800 3100
 Wire Wire Line
-	6150 3550 6400 3550
+	6100 3100 6350 3100
 Wire Wire Line
-	6400 3550 6400 3200
+	6350 3100 6350 2750
 $Sheet
 S 1350 900  1900 1300
@@
 F1 "USB2Serial.sch" 60
 $EndSheet
+$Sheet
+S 6850 1050 2350 1600
+U 58A32DD7
+F0 "Connectors" 60
+F1 "Connectors.sch" 60
+$EndSheet
+$Comp
+L SW_Push SW?
+U 1 1 58A33179
+P 3300 3200
+F 0 "SW?" H 3350 3300 50  0000 L CNN
+F 1 "SW_Push" H 3300 3140 50  0000 C CNN
+F 2 "" H 3300 3400 50  0000 C CNN
+F 3 "" H 3300 3400 50  0000 C CNN
+	1    3300 3200
+	0    1    1    0
+$EndComp
+Wire Wire Line
+	3800 3000 3300 3000
+$Comp
+L GND #PWR?
+U 1 1 58A3327D
+P 3300 3550
+F 0 "#PWR?" H 3300 3300 50  0001 C CNN
+F 1 "GND" H 3300 3400 50  0000 C CNN
+F 2 "" H 3300 3550 50  0000 C CNN
+F 3 "" H 3300 3550 50  0000 C CNN
+	1    3300 3550
+	1    0    0    -1
+$EndComp
+Wire Wire Line
+	3300 3550 3300 3400
+$Comp
+L R R?
+U 1 1 58A332A2
+P 3300 2700
+F 0 "R?" V 3380 2700 50  0000 C CNN
+F 1 "10k" V 3300 2700 50  0000 C CNN
+F 2 "" V 3230 2700 50  0000 C CNN
+F 3 "" H 3300 2700 50  0000 C CNN
+	1    3300 2700
+	1    0    0    -1
+$EndComp
+Wire Wire Line
+	3300 3000 3300 2850
+Wire Wire Line
+	3300 2550 3300 2400
+Text Label 3300 2400 0    60   ~ 0
+3.3V
+Text Label 6350 2750 0    60   ~ 0
+USB_RX
+Wire Wire Line
+	5600 3000 5850 3000
+Text Label 5850 3000 0    60   ~ 0
+TXD
+Wire Wire Line
+	5600 3200 6000 3200
+Wire Wire Line
+	5600 3300 6000 3300
+Wire Wire Line
+	5600 3400 6000 3400
+Wire Wire Line
+	5600 3500 6000 3500
+Wire Wire Line
+	5600 3600 6000 3600
+Wire Wire Line
+	3800 3100 3650 3100
+Wire Wire Line
+	3800 3200 3650 3200
+Wire Wire Line
+	3800 3300 3650 3300
+Wire Wire Line
+	3800 3400 3650 3400
+Wire Wire Line
+	3800 3500 3650 3500
+Wire Wire Line
+	3800 3600 3650 3600
+Wire Wire Line
+	3800 3700 3650 3700
+Text Label 3650 3700 0    60   ~ 0
+3.3V
+Text Label 3650 3300 0    60   ~ 0
+GPIO16
+Text Label 3650 3200 0    60   ~ 0
+CH_PD
+Text Label 3650 3100 0    60   ~ 0
+ADC
+Text Label 6000 3600 0    60   ~ 0
+GPIO15
+Text Label 6000 3500 0    60   ~ 0
+GPIO2
+Text Label 6000 3400 0    60   ~ 0
+GPIO0
+Text Label 6000 3300 0    60   ~ 0
+GPIO4/SDA
+Text Label 6000 3200 0    60   ~ 0
+GPIO5/SCL
+Text Label 5650 3100 0    60   ~ 0
+RXD
+Text Label 3650 3600 0    60   ~ 0
+GPIO13/MOSI
+Text Label 3650 3500 0    60   ~ 0
+GPIO12/MISO
+Text Label 3650 3400 0    60   ~ 0
+GPIO14/SCK
 $EndSCHEMATC

Commit message: 'rev1'
Parts:
- added U?: MCP9701T-E/TT, MCP9701T-E_TT:SOT95P237X112-3N, symbol MCP9701T-E/TT
- gave numbers to parts that had none: 4
Connections:
- wire segments 22 -> 26
Other:
- moved on the sheet: R1, SW1
Changed lines of the file:
@@
 LIBS:ESP8266
 LIBS:switches
+LIBS:ESP32-footprints-Shem-Lib
+LIBS:MCP9701T-E_TT
 LIBS:ESP8266_arduino-cache
 EELAYER 25 0
@@
 $EndDescr
 $Comp
-L ESP-12E U?
+L ESP-12E U1
 U 1 1 589B9F6E
 P 4700 3300
-F 0 "U?" H 4700 3200 50  0000 C CNN
+F 0 "U1" H 4700 3200 50  0000 C CNN
 F 1 "ESP-12E" H 4700 3400 50  0000 C CNN
 F 2 "" H 4700 3300 50  0001 C CNN
@@
 $EndComp
 $Comp
-L GND #PWR?
+L GND #PWR01
 U 1 1 589BA336
 P 5700 3900
-F 0 "#PWR?" H 5700 3650 50  0001 C CNN
+F 0 "#PWR01" H 5700 3650 50  0001 C CNN
 F 1 "GND" H 5700 3750 50  0000 C CNN
 F 2 "" H 5700 3900 50  0000 C CNN
@@
 	5700 3700 5700 3900
 $Comp
-L R R?
+L R R2
 U 1 1 589BA5F2
 P 5950 3100
-F 0 "R?" V 6030 3100 50  0000 C CNN
+F 0 "R2" V 6030 3100 50  0000 C CNN
 F 1 "1K" V 5950 3100 50  0000 C CNN
 F 2 "" V 5880 3100 50  0000 C CNN
@@
 $EndSheet
 $Comp
-L SW_Push SW?
+L SW_Push SW1
 U 1 1 58A33179
-P 3300 3200
-F 0 "SW?" H 3350 3300 50  0000 L CNN
-F 1 "SW_Push" H 3300 3140 50  0000 C CNN
-F 2 "" H 3300 3400 50  0000 C CNN
-F 3 "" H 3300 3400 50  0000 C CNN
-	1    3300 3200
+P 3200 3200
+F 0 "SW1" H 3250 3300 50  0000 L CNN
+F 1 "SW_Push" H 3200 3140 50  0000 C CNN
+F 2 "" H 3200 3400 50  0000 C CNN
+F 3 "" H 3200 3400 50  0000 C CNN
+	1    3200 3200
 	0    1    1    0
 $EndComp
 Wire Wire Line
-	3800 3000 3300 3000
-$Comp
-L GND #PWR?
+	3200 3000 3800 3000
+$Comp
+L GND #PWR02
 U 1 1 58A3327D
-P 3300 3550
-F 0 "#PWR?" H 3300 3300 50  0001 C CNN
-F 1 "GND" H 3300 3400 50  0000 C CNN
-F 2 "" H 3300 3550 50  0000 C CNN
-F 3 "" H 3300 3550 50  0000 C CNN
-	1    3300 3550
-	1    0    0    -1
-$EndComp
-Wire Wire Line
-	3300 3550 3300 3400
-$Comp
-L R R?
+P 3200 3550
+F 0 "#PWR02" H 3200 3300 50  0001 C CNN
+F 1 "GND" H 3200 3400 50  0000 C CNN
+F 2 "" H 3200 3550 50  0000 C CNN
+F 3 "" H 3200 3550 50  0000 C CNN
+	1    3200 3550
+	1    0    0    -1
+$EndComp
+Wire Wire Line
+	3200 3550 3200 3400
+$Comp
+L R R1
 U 1 1 58A332A2
-P 3300 2700
-F 0 "R?" V 3380 2700 50  0000 C CNN
-F 1 "10k" V 3300 2700 50  0000 C CNN
-F 2 "" V 3230 2700 50  0000 C CNN
-F 3 "" H 3300 2700 50  0000 C CNN
-	1    3300 2700
-	1    0    0    -1
-$EndComp
-Wire Wire Line
-	3300 3000 3300 2850
-Wire Wire Line
-	3300 2550 3300 2400
-Text Label 3300 2400 0    60   ~ 0
+P 3200 2700
+F 0 "R1" V 3280 2700 50  0000 C CNN
+F 1 "10k" V 3200 2700 50  0000 C CNN
+F 2 "" V 3130 2700 50  0000 C CNN
+F 3 "" H 3200 2700 50  0000 C CNN
+	1    3200 2700
+	1    0    0    -1
+$EndComp
+Wire Wire Line
+	3200 3000 3200 2850
+Wire Wire Line
+	3200 2550 3200 2400
+Text Label 3200 2400 0    60   ~ 0
 3.3V
 Text Label 6350 2750 0    60   ~ 0
@@
 TXD
 Wire Wire Line
-	5600 3200 6000 3200
-Wire Wire Line
-	5600 3300 6000 3300
-Wire Wire Line
-	5600 3400 6000 3400
-Wire Wire Line
-	5600 3500 6000 3500
-Wire Wire Line
-	5600 3600 6000 3600
-Wire Wire Line
-	3800 3100 3650 3100
-Wire Wire Line
-	3800 3200 3650 3200
-Wire Wire Line
-	3800 3300 3650 3300
-Wire Wire Line
-	3800 3400 3650 3400
-Wire Wire Line
-	3800 3500 3650 3500
-Wire Wire Line
-	3800 3600 3650 3600
+	5600 3200 6200 3200
+Wire Wire Line
+	5600 3300 6200 3300
+Wire Wire Line
+	5600 3400 6200 3400
+Wire Wire Line
+	5600 3500 7450 3500
+Wire Wire Line
+	5600 3600 6200 3600
+Wire Wire Line
+	3350 3100 3800 3100
+Wire Wire Line
+	3350 3200 3800 3200
+Wire Wire Line
+	3350 3300 3800 3300
+Wire Wire Line
+	3350 3400 3800 3400
+Wire Wire Line
+	3300 3500 3800 3500
+Wire Wire Line
+	3300 3600 3800 3600
 Wire Wire Line
 	3800 3700 3650 3700
 Text Label 3650 3700 0    60   ~ 0
 3.3V
-Text Label 3650 3300 0    60   ~ 0
+Text Label 3350 3300 0    60   ~ 0
 GPIO16
-Text Label 3650 3200 0    60   ~ 0
+Text Label 3350 3200 0    60   ~ 0
 CH_PD
-Text Label 3650 3100 0    60   ~ 0
+Text Label 3350 3100 0    60   ~ 0
 ADC
-Text Label 6000 3600 0    60   ~ 0
+Text Label 6200 3600 0    60   ~ 0
 GPIO15
-Text Label 6000 3500 0    60   ~ 0
+Text Label 6200 3500 0    60   ~ 0
 GPIO2
-Text Label 6000 3400 0    60   ~ 0
+Text Label 6200 3400 0    60   ~ 0
 GPIO0
-Text Label 6000 3300 0    60   ~ 0
+Text Label 6200 3300 0    60   ~ 0
 GPIO4/SDA
-Text Label 6000 3200 0    60   ~ 0
+Text Label 6200 3200 0    60   ~ 0
 GPIO5/SCL
 Text Label 5650 3100 0    60   ~ 0
 RXD
-Text Label 3650 3600 0    60   ~ 0
+Text Label 3300 3600 0    60   ~ 0
 GPIO13/MOSI
-Text Label 3650 3500 0    60   ~ 0
+Text Label 3300 3500 0    60   ~ 0
 GPIO12/MISO
-Text Label 3650 3400 0    60   ~ 0
+Text Label 3350 3400 0    60   ~ 0
 GPIO14/SCK
+$Comp
+L MCP9701T-E/TT U?
+U 1 1 58A3636F
+P 6750 4400
+F 0 "U?" H 6570 4611 50  0000 L CNN
+F 1 "MCP9701T-E/TT" H 6572 3835 50  0000 L CNN
+F 2 "MCP9701T-E_TT:SOT95P237X112-3N" H 6750 4400 50  0001 L CNN
+F 3 "Microchip MCP9701T-E/TT Temperature Sensor 3-Pin SOT-23, -40 - +125 degC" H 6750 4400 50  0001 L CNN
+F 4 "Good" H 6750 4400 50  0001 L CNN "Availability"
+F 5 "SOT-23-3 Microchip" H 6750 4400 50  0001 L CNN "Package"
+F 6 "Microchip" H 6750 4400 50  0001 L CNN "MF"
+F 7 "0.21 USD" H 6750 4400 50  0001 L CNN "Price"
+F 8 "MCP9701T-E/TT" H 6750 4400 50  0001 L CNN "MP"
+	1    6750 4400
+	1    0    0    -1
+$EndComp
+Wire Wire Line
+	7450 3500 7450 4500
+Text Label 5650 4500 0    60   ~ 0
+3.3V
+Wire Wire Line
+	5650 4500 6050 4500
+$Comp
+L GND #PWR?
+U 1 1 58A36768
+P 5850 4750
+F 0 "#PWR?" H 5850 4500 50  0001 C CNN
+F 1 "GND" H 5850 4600 50  0000 C CNN
+F 2 "" H 5850 4750 50  0000 C CNN
+F 3 "" H 5850 4750 50  0000 C CNN
+	1    5850 4750
+	1    0    0    -1
+$EndComp
+Wire Wire Line
+	6050 4600 5850 4600
+Wire Wire Line
+	5850 4600 5850 4750
 $EndSCHEMATC
