File: USB2Serial.sch (KiCad schematic (older format))
At the start: 3 parts

Commit message: 'rev1'
Parts:
- gave numbers to parts that had none: 3
Connections:
- net at P1.2 (D-), U3.3 (D+): no longer P1.3 (D+), U3.4 (D-)
- new net: P1.3 (D+), U3.4 (D-)
Changed lines of the file:
@@
 LIBS:ESP8266
 LIBS:switches
+LIBS:ESP32-footprints-Shem-Lib
+LIBS:MCP9701T-E_TT
 LIBS:ESP8266_arduino-cache
 EELAYER 25 0
@@
 $EndDescr
 $Comp
-L USB_OTG P?
+L USB_OTG P1
 U 1 1 589BE5FA
 P 2000 4150
-F 0 "P?" H 2325 4025 50  0000 C CNN
+F 0 "P1" H 2325 4025 50  0000 C CNN
 F 1 "USB_OTG" H 2000 4350 50  0000 C CNN
 F 2 "" V 1950 4050 50  0000 C CNN
@@
 VBUS
 $Comp
-L CP2104--USB/UART_BRIDGE U?
+L CP2104--USB/UART_BRIDGE U3
 U 1 1 58A323D1
 P 4400 2950
-F 0 "U?" H 4350 3450 50  0000 L CNN
+F 0 "U3" H 4350 3450 50  0000 L CNN
 F 1 "CP2104--USB/UART_BRIDGE" H 3850 3150 50  0000 L CIN
 F 2 "" H 4400 2750 50  0000 C CNN
@@
 	2550 3950 2550 3800
 Connection ~ 2550 3950
-Wire Wire Line
-	2300 4150 2900 4150
-Wire Wire Line
-	2900 4150 2900 4050
-Wire Wire Line
-	2900 4050 3300 4050
-Wire Wire Line
-	2300 4050 2750 4050
-Wire Wire Line
-	2750 4050 2750 4150
-Wire Wire Line
-	2750 4150 3300 4150
 Wire Wire Line
 	2650 1500 3300 1500
@@
 3.3V
 $Comp
-L GND #PWR?
+L GND #PWR05
 U 1 1 58A328F8
 P 2650 1950
-F 0 "#PWR?" H 2650 1700 50  0001 C CNN
+F 0 "#PWR05" H 2650 1700 50  0001 C CNN
 F 1 "GND" H 2650 1800 50  0000 C CNN
 F 2 "" H 2650 1950 50  0000 C CNN
@@
 $EndComp
 $Comp
-L C C?
+L C C3
 U 1 1 58A32914
 P 2650 1700
-F 0 "C?" H 2675 1800 50  0000 L CNN
+F 0 "C3" H 2675 1800 50  0000 L CNN
 F 1 "5uF" H 2675 1600 50  0000 L CNN
 F 2 "" H 2688 1550 50  0000 C CNN
@@
 	2650 1850 2650 1950
 $Comp
-L GND #PWR?
+L GND #PWR06
 U 1 1 58A329CC
 P 2900 1950
-F 0 "#PWR?" H 2900 1700 50  0001 C CNN
+F 0 "#PWR06" H 2900 1700 50  0001 C CNN
 F 1 "GND" H 2900 1800 50  0000 C CNN
 F 2 "" H 2900 1950 50  0000 C CNN
@@
 RTS
 $Comp
-L GND #PWR?
+L GND #PWR07
 U 1 1 58A32BC6
 P 2400 4600
-F 0 "#PWR?" H 2400 4350 50  0001 C CNN
+F 0 "#PWR07" H 2400 4350 50  0001 C CNN
 F 1 "GND" H 2400 4450 50  0000 C CNN
 F 2 "" H 2400 4600 50  0000 C CNN
@@
 Wire Wire Line
 	2400 4350 2400 4600
+Wire Wire Line
+	3300 4050 2300 4050
+Wire Wire Line
+	3300 4150 2300 4150
 $EndSCHEMATC
