File: regulation.sch (KiCad schematic (older format))
At the start: 4 parts

Commit message: 'rev1'
Parts:
- gave numbers to parts that had none: 4
Changed lines of the file:
@@
 LIBS:ESP8266
 LIBS:switches
+LIBS:ESP32-footprints-Shem-Lib
+LIBS:MCP9701T-E_TT
 LIBS:ESP8266_arduino-cache
 EELAYER 25 0
@@
 $EndDescr
 $Comp
-L MIC5524 U?
+L MIC5524 U2
 U 1 1 589BDF4A
 P 2700 2000
-F 0 "U?" H 2700 2350 50  0000 C CNN
+F 0 "U2" H 2700 2350 50  0000 C CNN
 F 1 "MIC5524" H 2700 2250 50  0000 C CNN
 F 2 "DFN-4:DFN-4" H 3100 1700 50  0001 L CIN
@@
 $EndComp
 $Comp
-L C C?
+L C C2
 U 1 1 589BE00C
 P 3300 2150
-F 0 "C?" H 3325 2250 50  0000 L CNN
+F 0 "C2" H 3325 2250 50  0000 L CNN
 F 1 "10uF" H 3325 2050 50  0000 L CNN
 F 2 "" H 3338 2000 50  0000 C CNN
@@
 $EndComp
 $Comp
-L GND #PWR?
+L GND #PWR03
 U 1 1 589BE161
 P 2700 2550
-F 0 "#PWR?" H 2700 2300 50  0001 C CNN
+F 0 "#PWR03" H 2700 2300 50  0001 C CNN
 F 1 "GND" H 2700 2400 50  0000 C CNN
 F 2 "" H 2700 2550 50  0000 C CNN
@@
 $EndComp
 $Comp
-L GND #PWR?
+L GND #PWR04
 U 1 1 58A0D21D
 P 1800 2750
-F 0 "#PWR?" H 1800 2500 50  0001 C CNN
+F 0 "#PWR04" H 1800 2500 50  0001 C CNN
 F 1 "GND" H 1800 2600 50  0000 C CNN
 F 2 "" H 1800 2750 50  0000 C CNN
@@
 VBUS
 $Comp
-L C C?
+L C C1
 U 1 1 58A0D54C
 P 1800 2300
-F 0 "C?" H 1825 2400 50  0000 L CNN
+F 0 "C1" H 1825 2400 50  0000 L CNN
 F 1 "10uF" H 1825 2200 50  0000 L CNN
 F 2 "" H 1838 2150 50  0000 C CNN
@@
 3.3V
 $Comp
-L R R?
+L R R3
 U 1 1 58A33F9D
 P 2000 2100
-F 0 "R?" V 2080 2100 50  0000 C CNN
+F 0 "R3" V 2080 2100 50  0000 C CNN
 F 1 "10k" V 2000 2100 50  0000 C CNN
 F 2 "" V 1930 2100 50  0000 C CNN
